File: connectors.kicad_sch (KiCad schematic)
At the start: 14 parts, among them J1 SM06B-SRSS-TB_LF__SN_, J2 SM06B-SRSS-TB_LF__SN_, J4 SM08B-SRSS-TB_LF__SN_, J5 Debug Header, J6 UJ20-C-H-G-SMT-1-P16-TR, Q2 SS8050

Commit message: Finished system overview
Parts:
- removed J1, J2: SM06B-SRSS-TB_LF__SN_, KSE_connector:JST_SM06B-SRSS-TB_LF__SN_, symbol KSE_connectors:SM06B-SRSS-TB_LF__SN_
- removed J4: SM08B-SRSS-TB_LF__SN_, KSE_connector:JST_SM08B-SRSS-TB_LF__SN_, symbol KSE_connectors:SM08B-SRSS-TB_LF__SN_
- removed J5: Debug Header, Connector_PinHeader_2.54mm:PinHeader_2x03_P2.54mm_Vertical, symbol Connector_Generic:Conn_02x03_Odd_Even
- removed J6: UJ20-C-H-G-SMT-1-P16-TR, KSE_connector:SAMESKY_UJ20-C-H-G-SMT-1-P16-TR, symbol KSE_connectors:UJ20-C-H-G-SMT-1-P16-TR
- removed Q2: SS8050, Package_TO_SOT_SMD:SOT-23, symbol Transistor_BJT:SS8050
- removed R1: 75k, Resistor_SMD:R_0603_1608Metric_Pad0.98x0.95mm_HandSolder, symbol Device:R_Small
- removed R10, R7: 4.7k, Resistor_SMD:R_0603_1608Metric_Pad0.98x0.95mm_HandSolder, symbol Device:R_Small
- removed R15, R9: 5.1k, Resistor_SMD:R_0805_2012Metric_Pad1.20x1.40mm_HandSolder, symbol Device:R
- removed R2, R3: 10k, Resistor_SMD:R_0603_1608Metric_Pad0.98x0.95mm_HandSolder, symbol Device:R_Small
- removed R4: 1k, Resistor_SMD:R_0603_1608Metric_Pad0.98x0.95mm_HandSolder, symbol Device:R_Small
Connections:
- no-connect marks 3 -> 0
Other:
- note removed: "+VBAT"
- note removed: "-VBAT"
- note removed: "3A Sink"
- note removed: "4-in-1 ESC Interface (Betaflight)"
- note removed: "CURR"
- note removed: "DESIGN NOTE: ESC signals can be: - DSHOT - Multishot - Oneshot - PWM"
- note removed: "DESIGN NOTE: SBUS to UART Inverter"
- note removed: "DESIGN NOTE: Volage divider ratio: 11.77 : 1"
- note removed: "DOUBLE CHECK CONNECTOR PIN-OUT!"
- note removed: "ESC Connector"
- note removed: "GPS+COMPASS Connctor"
- note removed: "M1"
- note removed: "M2"
- note removed: "M3"
- note removed: "M4"
- note removed: "MCU Debug Header"
- note removed: "PGND"
- note removed: "Receiver"
- note removed: "S.BUS"
- note removed: "SGND"
- note removed: "TELE"
- note removed: "Transmitter"
- note removed: "USB-C INTERFACE"
- note removed: "VCC"
- note removed: "VTX Connector"
- note removed: "VTX Interface (DJI 04 AIR)"
